Commit message: add lidar

File: description/gazebo_control.xacro (robot description, xacro)
@@ -18,4 +18,7 @@
             <publish_wheel_tf>true</publish_wheel_tf>
         </plugin>
+        <plugin name="joint_state_publisher" filename="libgazebo_ros_joint_state_publisher.so">
+            <jointName>left_wheel,right_wheel</jointName>
+        </plugin>
     </gazebo>
 </robot>

File: description/robot.urdf.xacro (robot description, xacro)
@@ -12,4 +12,6 @@
     <xacro:include filename="camera.xacro" />
     <!-- <xacro:include filename="depth_camera.xacro" /> -->
+    <xacro:include filename="lidar.xacro" />
+    <!-- <xacro:include filename="depth_camera.xacro" /> -->
     <xacro:include filename="face.xacro" />
 </robot>

File: description/robot_core.xacro (robot description, xacro)
@@ -10,4 +10,5 @@
     <xacro:property name="wheel_mass" value="0.05"/>
     <xacro:property name="wheel_offset_x" value="0.226"/>
+    <xacro:property name="wheel_offset_h" value="-0.116"/>
     <xacro:property name="wheel_offset_y" value="0.1485"/>
     <xacro:property name="wheel_offset_z" value="0.01"/>
@@ -121,5 +122,5 @@
         <parent link="base_link"/>
         <child link="back_left_wheel"/>
-        <origin xyz="0 ${wheel_offset_y} 0" rpy="-${pi/2} 0 0" />
+        <origin xyz="${wheel_offset_h} ${wheel_offset_y} 0" rpy="-${pi/2} 0 0" />
         <axis xyz="0 0 1"/>
     </joint>
@@ -147,5 +148,5 @@
         <parent link="base_link"/>
         <child link="back_right_wheel"/>
-        <origin xyz="0 ${-wheel_offset_y} 0" rpy="${pi/2} 0 0" />
+        <origin xyz="${wheel_offset_h} ${-wheel_offset_y} 0" rpy="${pi/2} 0 0" />
         <axis xyz="0 0 -1"/>
     </joint>
