Commit message: Camera moved

File: description/camera.xacro (robot description, xacro)
@@ -4,5 +4,5 @@
         <parent link="chassis"/>
         <child link="camera_link"/>
-        <origin xyz="0.276 0 0.181" rpy="0 0.18 0"/>
+        <origin xyz="${chassis_length} 0 ${chassis_height}"/>
     </joint>
     <link name="camera_link">

Commit message: Revert "Camera moved"
This reverts commit e40672751ae4361bc97b7e0ab74e184f8c9fbec0.

erase

File: description/camera.xacro (robot description, xacro)
@@ -4,5 +4,5 @@
         <parent link="chassis"/>
         <child link="camera_link"/>
-        <origin xyz="${chassis_length} 0 ${chassis_height}"/>
+        <origin xyz="0.276 0 0.181" rpy="0 0.18 0"/>
     </joint>
     <link name="camera_link">

Commit message: Update camera.xacro
Move Camera

File: description/camera.xacro (robot description, xacro)
@@ -4,5 +4,5 @@
         <parent link="chassis"/>
         <child link="camera_link"/>
-        <origin xyz="0.276 0 0.181" rpy="0 0.18 0"/>
+        <origin xyz="${chassis_length} 0 ${chassis_height}" rpy="0 0.18 0"/>
     </joint>
     <link name="camera_link">

Commit message: Changed camera tilt. Works in Gazebo

File: description/camera.xacro (robot description, xacro)
@@ -4,5 +4,5 @@
         <parent link="chassis"/>
         <child link="camera_link"/>
-        <origin xyz="${chassis_length} 0 ${chassis_height}" rpy="0 0.18 0"/>
+        <origin xyz="${chassis_length} 0 ${chassis_height}" rpy="0 0.5 0"/>
     </joint>
     <link name="camera_link">
